Commit message: Organize integrated robot and Gazebo tools under simulation

File: simulation/robot_description/sensor_rack_piper/sensor_rack_piper.urdf (robot description, URDF)
Before this commit: robot sensor_rack_piper, 74 links, 73 joints
Links:
- link base_link: geometry collision box size=0.04 0.04 0.04; collision box size=0.04 0.04 0.04
- link camera_link: geometry collision box size=0.02557999999 0.08990450611 0.02499995771; collision box size=6.6e-05 0.08319 0.01539
- link g2_link: geometry collision box size=0.0737 0.0737 0.0205; collision box size=0.08135 0.0782820323 0.0205
- link mid360_link: geometry collision box size=0.073 0.065 0.039576; visual mesh filename=../../../HW/URDF/sensor_rack_description/meshes/mid360_link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 scale=1 1 1
- link piper_base_link: geometry collision mesh filename=../../../HW/URDF/piper/meshes/base_link.stl; visual mesh filename=../../../HW/URDF/piper/meshes/dae/base_link.dae
- link piper_flange_link: geometry collision mesh filename=../../../HW/URDF/piper/meshes/flange.stl; visual mesh filename=../../../HW/URDF/piper/meshes/dae/flange.dae
- link piper_gripper_base: geometry collision mesh filename=../../../HW/URDF/piper/meshes/gripper_base.stl; visual mesh filename=../../../HW/URDF/piper/meshes/dae/gripper_base.dae
- link piper_gripper_link1: geometry collision mesh filename=../../../HW/URDF/piper/meshes/gripper_link1.stl; visual mesh filename=../../../HW/URDF/piper/meshes/dae/gripper_link1.dae
- link piper_gripper_link2: geometry collision mesh filename=../../../HW/URDF/piper/meshes/gripper_link2.stl; visual mesh filename=../../../HW/URDF/piper/meshes/dae/gripper_link2.dae
- link piper_link1: geometry collision mesh filename=../../../HW/URDF/piper/meshes/link1.stl; visual mesh filename=../../../HW/URDF/piper/meshes/dae/link1.dae
- link piper_link2: geometry collision mesh filename=../../../HW/URDF/piper/meshes/link2.stl; visual mesh filename=../../../HW/URDF/piper/meshes/dae/link2.dae
- link piper_link3: geometry collision mesh filename=../../../HW/URDF/piper/meshes/link3.stl; visual mesh filename=../../../HW/URDF/piper/meshes/dae/link3.dae
- link piper_link4: geometry collision mesh filename=../../../HW/URDF/piper/meshes/link4.stl; visual mesh filename=../../../HW/URDF/piper/meshes/dae/link4.dae
- link piper_link5: geometry collision mesh filename=../../../HW/URDF/piper/meshes/link5.stl; visual mesh filename=../../../HW/URDF/piper/meshes/dae/link5.dae
- link piper_link6: geometry collision mesh filename=../../../HW/URDF/piper/meshes/link6.stl; visual mesh filename=../../../HW/URDF/piper/meshes/dae/link6.dae

File: simulation/robot_description/sensor_rack_piper/sensor_rack_piper_gazebo.urdf (robot description, URDF)
Before this commit: robot tracer_sensor_rack_piper, 85 links, 84 joints
Links:
- removed link fl_castor_link
- removed link fl_wheel_link
- removed link fr_castor_link
- removed link fr_wheel_link
- removed link inertial_link
- removed link left_wheel_link
- removed link rack_base_link
- removed link right_wheel_link
- removed link rl_castor_link
- removed link rl_wheel_link
- removed link rr_castor_link
- removed link rr_wheel_link
- link base_link: mass None -> 15.85407974; geometry collision box size=0.04 0.04 0.04; collision box size=0.04 0.04 0.04
- link camera_link: geometry collision box size=0.02557999999 0.08990450611 0.02499995771; collision box size=6.6e-05 0.08319 0.01539
- link g2_link: geometry collision box size=0.0737 0.0737 0.0205; collision box size=0.08135 0.0782820323 0.0205
- link mid360_link: geometry collision box size=0.073 0.065 0.039576; visual mesh filename=../../../HW/URDF/sensor_rack_description/meshes/mid360_link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 scale=1 1 1
- link piper_base_link: geometry collision mesh filename=../../../HW/URDF/piper/meshes/base_link.stl; visual mesh filename=../../../HW/URDF/piper/meshes/dae/base_link.dae
- link piper_flange_link: geometry collision mesh filename=../../../HW/URDF/piper/meshes/flange.stl; visual mesh filename=../../../HW/URDF/piper/meshes/dae/flange.dae
- link piper_gripper_base: geometry collision mesh filename=../../../HW/URDF/piper/meshes/gripper_base.stl; visual mesh filename=../../../HW/URDF/piper/meshes/dae/gripper_base.dae
- link piper_gripper_link1: geometry collision mesh filename=../../../HW/URDF/piper/meshes/gripper_link1.stl; visual mesh filename=../../../HW/URDF/piper/meshes/dae/gripper_link1.dae
- link piper_gripper_link2: geometry collision mesh filename=../../../HW/URDF/piper/meshes/gripper_link2.stl; visual mesh filename=../../../HW/URDF/piper/meshes/dae/gripper_link2.dae
- link piper_link1: geometry collision mesh filename=../../../HW/URDF/piper/meshes/link1.stl; visual mesh filename=../../../HW/URDF/piper/meshes/dae/link1.dae
- link piper_link2: geometry collision mesh filename=../../../HW/URDF/piper/meshes/link2.stl; visual mesh filename=../../../HW/URDF/piper/meshes/dae/link2.dae
- link piper_link3: geometry collision mesh filename=../../../HW/URDF/piper/meshes/link3.stl; visual mesh filename=../../../HW/URDF/piper/meshes/dae/link3.dae
- link piper_link4: geometry collision mesh filename=../../../HW/URDF/piper/meshes/link4.stl; visual mesh filename=../../../HW/URDF/piper/meshes/dae/link4.dae
- link piper_link5: geometry collision mesh filename=../../../HW/URDF/piper/meshes/link5.stl; visual mesh filename=../../../HW/URDF/piper/meshes/dae/link5.dae
- link piper_link6: geometry collision mesh filename=../../../HW/URDF/piper/meshes/link6.stl; visual mesh filename=../../../HW/URDF/piper/meshes/dae/link6.dae
Joints:
- removed joint fl_castor_wheel
- removed joint fl_wheel
- removed joint fr_castor_wheel
- removed joint fr_wheel
- removed joint inertial_joint
- removed joint left_wheel
- removed joint right_wheel
- removed joint rl_castor_wheel
- removed joint rl_wheel
- removed joint rr_castor_wheel
- removed joint rr_wheel
- removed joint tracer_to_rack
- joint cad_2D_LiDARMount_1_joint: parent rack_base_link -> base_link
- joint cad_3D_LiDAR_Camera_mount_1_joint: parent rack_base_link -> base_link
- joint cad_D435f_Solid_v1_1_joint: parent rack_base_link -> base_link
- joint cad_Manipulator_mount_1_joint: parent rack_base_link -> base_link
- joint cad_YDLIDAR_G2_base_1_Base_1_joint: parent rack_base_link -> base_link
- joint cad_YDLIDAR_G2_base_1_joint: parent rack_base_link -> base_link
- joint cad_YDLIDAR_G2_top_1_TOP_1_joint: parent rack_base_link -> base_link
- joint cad_YDLIDAR_G2_top_1_joint: parent rack_base_link -> base_link
- joint cad____1_1_OUT_SHELL_1_joint: parent rack_base_link -> base_link
- joint cad_bracket_10_joint: parent rack_base_link -> base_link
- joint cad_bracket_11_joint: parent rack_base_link -> base_link
- joint cad_bracket_12_joint: parent rack_base_link -> base_link
- joint cad_bracket_13_joint: parent rack_base_link -> base_link
- joint cad_bracket_14_joint: parent rack_base_link -> base_link
- joint cad_bracket_15_joint: parent rack_base_link -> base_link
- joint cad_bracket_16_joint: parent rack_base_link -> base_link
- joint cad_bracket_17_joint: parent rack_base_link -> base_link
- joint cad_bracket_18_joint: parent rack_base_link -> base_link
- joint cad_bracket_1_joint: parent rack_base_link -> base_link
- joint cad_bracket_21_joint: parent rack_base_link -> base_link
- joint cad_bracket_22_joint: parent rack_base_link -> base_link
- joint cad_bracket_23_joint: parent rack_base_link -> base_link
- joint cad_bracket_24_joint: parent rack_base_link -> base_link
- joint cad_bracket_2_joint: parent rack_base_link -> base_link
- joint cad_bracket_3_joint: parent rack_base_link -> base_link
- joint cad_bracket_4_joint: parent rack_base_link -> base_link
- joint cad_bracket_5_joint: parent rack_base_link -> base_link
- joint cad_bracket_6_joint: parent rack_base_link -> base_link
- joint cad_bracket_7_joint: parent rack_base_link -> base_link
- joint cad_bracket_8_joint: parent rack_base_link -> base_link
- joint cad_bracket_9_joint: parent rack_base_link -> base_link
- joint cad_component_51_joint: parent rack_base_link -> base_link
- joint cad_mid_360s_axis_1_joint: parent rack_base_link -> base_link
- joint cad_profiles_250mm_1_joint: parent rack_base_link -> base_link
- joint cad_profiles_250mm_2_joint: parent rack_base_link -> base_link
- joint cad_profiles_250mm_3_joint: parent rack_base_link -> base_link
- joint cad_profiles_250mm_4_joint: parent rack_base_link -> base_link
- joint cad_profiles_250mm_5_joint: parent rack_base_link -> base_link
- joint cad_profiles_320mm_1_joint: parent rack_base_link -> base_link
- joint cad_profiles_320mm_2_joint: parent rack_base_link -> base_link
- joint cad_profiles_320mm_3_joint: parent rack_base_link -> base_link
- joint cad_profiles_320mm_4_joint: parent rack_base_link -> base_link
- joint cad_profiles_390mm_1_joint: parent rack_base_link -> base_link
- joint cad_profiles_390mm_2_joint: parent rack_base_link -> base_link
- joint cad_profiles_390mm_3_joint: parent rack_base_link -> base_link
- joint cad_profiles_390mm_4_joint: parent rack_base_link -> base_link
- joint cad_profiles_470mm_1_joint: parent rack_base_link -> base_link
- joint cad_profiles_470mm_2_joint: parent rack_base_link -> base_link
- joint cad_profiles_500mm_1_joint: parent rack_base_link -> base_link
- joint cad_profiles_500mm_2_joint: parent rack_base_link -> base_link
- joint cad_profiles_500mm_3_joint: parent rack_base_link -> base_link
- joint cad_profiles_500mm_4_joint: parent rack_base_link -> base_link
- joint cad_profiles_500mm_5_joint: parent rack_base_link -> base_link
- joint cad_profiles_500mm_6_joint: parent rack_base_link -> base_link
- joint camera_link_joint: parent rack_base_link -> base_link
- joint g2_link_joint: parent rack_base_link -> base_link
- joint mid360_link_joint: parent rack_base_link -> base_link

File: simulation/robot_description/tracer_sensor_rack_piper.urdf (robot description, URDF)
Before this commit: robot tracer_sensor_rack_piper, 86 links, 85 joints
Links:
- link base_link: geometry collision mesh filename=../../HW/URDF/tracer/meshes/tracer_base_link_no_wheel.dae; visual mesh filename=../../HW/URDF/tracer/meshes/tracer_base_link_no_wheel.dae
- link camera_link: geometry collision box size=0.02557999999 0.08990450611 0.02499995771; collision box size=6.6e-05 0.08319 0.01539
- link fl_castor_link: geometry visual mesh filename=../../HW/URDF/tracer/meshes/castor_joint.dae
- link fl_wheel_link: geometry collision mesh filename=../../HW/URDF/tracer/meshes/castor.dae; visual mesh filename=../../HW/URDF/tracer/meshes/castor.dae
- link fr_castor_link: geometry visual mesh filename=../../HW/URDF/tracer/meshes/castor_joint.dae
- link fr_wheel_link: geometry collision mesh filename=../../HW/URDF/tracer/meshes/castor.dae; visual mesh filename=../../HW/URDF/tracer/meshes/castor.dae
- link g2_link: geometry collision box size=0.0737 0.0737 0.0205; collision box size=0.08135 0.0782820323 0.0205
- link left_wheel_link: geometry collision mesh filename=../../HW/URDF/tracer/meshes/tracer_wheel.dae; visual mesh filename=../../HW/URDF/tracer/meshes/tracer_wheel.dae
- link mid360_link: geometry collision box size=0.073 0.065 0.039576; visual mesh filename=../../HW/URDF/sensor_rack_description/meshes/mid360_link.stl scale=1 1 1
- link piper_base_link: geometry collision mesh filename=../../HW/URDF/piper/meshes/base_link.stl; visual mesh filename=../../HW/URDF/piper/meshes/dae/base_link.dae
- link piper_flange_link: geometry collision mesh filename=../../HW/URDF/piper/meshes/flange.stl; visual mesh filename=../../HW/URDF/piper/meshes/dae/flange.dae
- link piper_gripper_base: geometry collision mesh filename=../../HW/URDF/piper/meshes/gripper_base.stl; visual mesh filename=../../HW/URDF/piper/meshes/dae/gripper_base.dae
- link piper_gripper_link1: geometry collision mesh filename=../../HW/URDF/piper/meshes/gripper_link1.stl; visual mesh filename=../../HW/URDF/piper/meshes/dae/gripper_link1.dae
- link piper_gripper_link2: geometry collision mesh filename=../../HW/URDF/piper/meshes/gripper_link2.stl; visual mesh filename=../../HW/URDF/piper/meshes/dae/gripper_link2.dae
- link piper_link1: geometry collision mesh filename=../../HW/URDF/piper/meshes/link1.stl; visual mesh filename=../../HW/URDF/piper/meshes/dae/link1.dae
- link piper_link2: geometry collision mesh filename=../../HW/URDF/piper/meshes/link2.stl; visual mesh filename=../../HW/URDF/piper/meshes/dae/link2.dae
- link piper_link3: geometry collision mesh filename=../../HW/URDF/piper/meshes/link3.stl; visual mesh filename=../../HW/URDF/piper/meshes/dae/link3.dae
- link piper_link4: geometry collision mesh filename=../../HW/URDF/piper/meshes/link4.stl; visual mesh filename=../../HW/URDF/piper/meshes/dae/link4.dae
- link piper_link5: geometry collision mesh filename=../../HW/URDF/piper/meshes/link5.stl; visual mesh filename=../../HW/URDF/piper/meshes/dae/link5.dae
- link piper_link6: geometry collision mesh filename=../../HW/URDF/piper/meshes/link6.stl; visual mesh filename=../../HW/URDF/piper/meshes/dae/link6.dae
- link rack_base_link: geometry collision box size=0.04 0.04 0.04; collision box size=0.04 0.04 0.04
- link right_wheel_link: geometry collision mesh filename=../../HW/URDF/tracer/meshes/tracer_wheel.dae; visual mesh filename=../../HW/URDF/tracer/meshes/tracer_wheel.dae
- link rl_castor_link: geometry visual mesh filename=../../HW/URDF/tracer/meshes/castor_joint.dae
- link rl_wheel_link: geometry collision mesh filename=../../HW/URDF/tracer/meshes/castor.dae; visual mesh filename=../../HW/URDF/tracer/meshes/castor.dae
- link rr_castor_link: geometry visual mesh filename=../../HW/URDF/tracer/meshes/castor_joint.dae
- link rr_wheel_link: geometry collision mesh filename=../../HW/URDF/tracer/meshes/castor.dae; visual mesh filename=../../HW/URDF/tracer/meshes/castor.dae
