Commit message: Organize integrated robot and Gazebo tools under simulation

File: simulation/robot_description/tracer_sensor_rack_piper_gazebo.urdf (robot description, URDF)
Before this commit: robot sensor_rack_piper, 73 links, 72 joints
Links:
- added link fl_castor_link, mass 1; visual mesh filename=../../HW/URDF/tracer/meshes/castor_joint.dae
- added link fl_wheel_link, mass 1; collision mesh filename=../../HW/URDF/tracer/meshes/castor.dae; visual mesh filename=../../HW/URDF/tracer/meshes/castor.dae
- added link fr_castor_link, mass 1; visual mesh filename=../../HW/URDF/tracer/meshes/castor_joint.dae
- added link fr_wheel_link, mass 1; collision mesh filename=../../HW/URDF/tracer/meshes/castor.dae; visual mesh filename=../../HW/URDF/tracer/meshes/castor.dae
- added link inertial_link, mass 132.3898489950015
- added link left_wheel_link, mass 6; collision mesh filename=../../HW/URDF/tracer/meshes/tracer_wheel.dae; visual mesh filename=../../HW/URDF/tracer/meshes/tracer_wheel.dae
- added link rack_base_link, mass 15.85407974; collision box size=0.04 0.04 0.04; collision box size=0.04 0.04 0.04
- added link right_wheel_link, mass 6; collision mesh filename=../../HW/URDF/tracer/meshes/tracer_wheel.dae; visual mesh filename=../../HW/URDF/tracer/meshes/tracer_wheel.dae
- added link rl_castor_link, mass 1; visual mesh filename=../../HW/URDF/tracer/meshes/castor_joint.dae
- added link rl_wheel_link, mass 1; collision mesh filename=../../HW/URDF/tracer/meshes/castor.dae; visual mesh filename=../../HW/URDF/tracer/meshes/castor.dae
- added link rr_castor_link, mass 1; visual mesh filename=../../HW/URDF/tracer/meshes/castor_joint.dae
- added link rr_wheel_link, mass 1; collision mesh filename=../../HW/URDF/tracer/meshes/castor.dae; visual mesh filename=../../HW/URDF/tracer/meshes/castor.dae
- link base_link: mass 15.85407974 -> None; geometry collision mesh filename=../../HW/URDF/tracer/meshes/tracer_base_link_no_wheel.dae; visual mesh filename=../../HW/URDF/tracer/meshes/tracer_base_link_no_wheel.dae
- link camera_link: geometry collision box size=0.02557999999 0.08990450611 0.02499995771; collision box size=6.6e-05 0.08319 0.01539
- link g2_link: geometry collision box size=0.0737 0.0737 0.0205; collision box size=0.08135 0.0782820323 0.0205
- link mid360_link: geometry collision box size=0.073 0.065 0.039576; visual mesh filename=../../HW/URDF/sensor_rack_description/meshes/mid360_link.stl scale=1 1 1
- link piper_base_link: geometry collision mesh filename=../../HW/URDF/piper/meshes/base_link.stl; visual mesh filename=../../HW/URDF/piper/meshes/dae/base_link.dae
- link piper_flange_link: geometry collision mesh filename=../../HW/URDF/piper/meshes/flange.stl; visual mesh filename=../../HW/URDF/piper/meshes/dae/flange.dae
- link piper_gripper_base: geometry collision mesh filename=../../HW/URDF/piper/meshes/gripper_base.stl; visual mesh filename=../../HW/URDF/piper/meshes/dae/gripper_base.dae
- link piper_gripper_link1: geometry collision mesh filename=../../HW/URDF/piper/meshes/gripper_link1.stl; visual mesh filename=../../HW/URDF/piper/meshes/dae/gripper_link1.dae
- link piper_gripper_link2: geometry collision mesh filename=../../HW/URDF/piper/meshes/gripper_link2.stl; visual mesh filename=../../HW/URDF/piper/meshes/dae/gripper_link2.dae
- link piper_link1: geometry collision mesh filename=../../HW/URDF/piper/meshes/link1.stl; visual mesh filename=../../HW/URDF/piper/meshes/dae/link1.dae
- link piper_link2: geometry collision mesh filename=../../HW/URDF/piper/meshes/link2.stl; visual mesh filename=../../HW/URDF/piper/meshes/dae/link2.dae
- link piper_link3: geometry collision mesh filename=../../HW/URDF/piper/meshes/link3.stl; visual mesh filename=../../HW/URDF/piper/meshes/dae/link3.dae
- link piper_link4: geometry collision mesh filename=../../HW/URDF/piper/meshes/link4.stl; visual mesh filename=../../HW/URDF/piper/meshes/dae/link4.dae
- link piper_link5: geometry collision mesh filename=../../HW/URDF/piper/meshes/link5.stl; visual mesh filename=../../HW/URDF/piper/meshes/dae/link5.dae
- link piper_link6: geometry collision mesh filename=../../HW/URDF/piper/meshes/link6.stl; visual mesh filename=../../HW/URDF/piper/meshes/dae/link6.dae
Joints:
- added joint fl_castor_wheel: type continuous, parent base_link, child fl_castor_link, origin xyz=0.18955 0.17 -0.0380886 rpy=-1.57 0 0, axis 0 1 0
- added joint fl_wheel: type continuous, parent fl_castor_link, child fl_wheel_link, origin xyz=-0.0218084 0.067 0 rpy=0 0 0, axis 0 0 1
- added joint fr_castor_wheel: type continuous, parent base_link, child fr_castor_link, origin xyz=0.18955 -0.17 -0.0380886 rpy=-1.57 0 0, axis 0 1 0
- added joint fr_wheel: type continuous, parent fr_castor_link, child fr_wheel_link, origin xyz=-0.0218084 0.067 0 rpy=0 0 0, axis 0 0 1
- added joint inertial_joint: type fixed, parent base_link, child inertial_link, origin xyz=0 0 0 rpy=0 0 0
- added joint left_wheel: type continuous, parent base_link, child left_wheel_link, origin xyz=0 0.17 -0.082 rpy=3.14 0 0, axis 0 1 0
- added joint right_wheel: type continuous, parent base_link, child right_wheel_link, origin xyz=0 -0.17 -0.082 rpy=0 0 0, axis 0 1 0
- added joint rl_castor_wheel: type continuous, parent base_link, child rl_castor_link, origin xyz=-0.18955 0.17 -0.0380886 rpy=-1.57 0 0, axis 0 1 0
- added joint rl_wheel: type continuous, parent rl_castor_link, child rl_wheel_link, origin xyz=-0.0218084 0.067 0 rpy=0 0 0, axis 0 0 1
- added joint rr_castor_wheel: type continuous, parent base_link, child rr_castor_link, origin xyz=-0.18955 -0.17 -0.0380886 rpy=-1.57 0 0, axis 0 1 0
- added joint rr_wheel: type continuous, parent rr_castor_link, child rr_wheel_link, origin xyz=-0.0218084 0.067 0 rpy=0 0 0, axis 0 0 1
- added joint tracer_to_rack: type fixed, parent base_link, child rack_base_link, origin xyz=0 0 0.01611 rpy=0 0 0
- joint cad_2D_LiDARMount_1_joint: parent base_link -> rack_base_link
- joint cad_3D_LiDAR_Camera_mount_1_joint: parent base_link -> rack_base_link
- joint cad_D435f_Solid_v1_1_joint: parent base_link -> rack_base_link
- joint cad_Manipulator_mount_1_joint: parent base_link -> rack_base_link
- joint cad_YDLIDAR_G2_base_1_Base_1_joint: parent base_link -> rack_base_link
- joint cad_YDLIDAR_G2_base_1_joint: parent base_link -> rack_base_link
- joint cad_YDLIDAR_G2_top_1_TOP_1_joint: parent base_link -> rack_base_link
- joint cad_YDLIDAR_G2_top_1_joint: parent base_link -> rack_base_link
- joint cad____1_1_OUT_SHELL_1_joint: parent base_link -> rack_base_link
- joint cad_bracket_10_joint: parent base_link -> rack_base_link
- joint cad_bracket_11_joint: parent base_link -> rack_base_link
- joint cad_bracket_12_joint: parent base_link -> rack_base_link
- joint cad_bracket_13_joint: parent base_link -> rack_base_link
- joint cad_bracket_14_joint: parent base_link -> rack_base_link
- joint cad_bracket_15_joint: parent base_link -> rack_base_link
- joint cad_bracket_16_joint: parent base_link -> rack_base_link
- joint cad_bracket_17_joint: parent base_link -> rack_base_link
- joint cad_bracket_18_joint: parent base_link -> rack_base_link
- joint cad_bracket_1_joint: parent base_link -> rack_base_link
- joint cad_bracket_21_joint: parent base_link -> rack_base_link
- joint cad_bracket_22_joint: parent base_link -> rack_base_link
- joint cad_bracket_23_joint: parent base_link -> rack_base_link
- joint cad_bracket_24_joint: parent base_link -> rack_base_link
- joint cad_bracket_2_joint: parent base_link -> rack_base_link
- joint cad_bracket_3_joint: parent base_link -> rack_base_link
- joint cad_bracket_4_joint: parent base_link -> rack_base_link
- joint cad_bracket_5_joint: parent base_link -> rack_base_link
- joint cad_bracket_6_joint: parent base_link -> rack_base_link
- joint cad_bracket_7_joint: parent base_link -> rack_base_link
- joint cad_bracket_8_joint: parent base_link -> rack_base_link
- joint cad_bracket_9_joint: parent base_link -> rack_base_link
- joint cad_component_51_joint: parent base_link -> rack_base_link
- joint cad_mid_360s_axis_1_joint: parent base_link -> rack_base_link
- joint cad_profiles_250mm_1_joint: parent base_link -> rack_base_link
- joint cad_profiles_250mm_2_joint: parent base_link -> rack_base_link
- joint cad_profiles_250mm_3_joint: parent base_link -> rack_base_link
- joint cad_profiles_250mm_4_joint: parent base_link -> rack_base_link
- joint cad_profiles_250mm_5_joint: parent base_link -> rack_base_link
- joint cad_profiles_320mm_1_joint: parent base_link -> rack_base_link
- joint cad_profiles_320mm_2_joint: parent base_link -> rack_base_link
- joint cad_profiles_320mm_3_joint: parent base_link -> rack_base_link
- joint cad_profiles_320mm_4_joint: parent base_link -> rack_base_link
- joint cad_profiles_390mm_1_joint: parent base_link -> rack_base_link
- joint cad_profiles_390mm_2_joint: parent base_link -> rack_base_link
- joint cad_profiles_390mm_3_joint: parent base_link -> rack_base_link
- joint cad_profiles_390mm_4_joint: parent base_link -> rack_base_link
- joint cad_profiles_470mm_1_joint: parent base_link -> rack_base_link
- joint cad_profiles_470mm_2_joint: parent base_link -> rack_base_link
- joint cad_profiles_500mm_1_joint: parent base_link -> rack_base_link
- joint cad_profiles_500mm_2_joint: parent base_link -> rack_base_link
- joint cad_profiles_500mm_3_joint: parent base_link -> rack_base_link
- joint cad_profiles_500mm_4_joint: parent base_link -> rack_base_link
- joint cad_profiles_500mm_5_joint: parent base_link -> rack_base_link
- joint cad_profiles_500mm_6_joint: parent base_link -> rack_base_link
- joint camera_link_joint: parent base_link -> rack_base_link
- joint g2_link_joint: parent base_link -> rack_base_link
- joint mid360_link_joint: parent base_link -> rack_base_link
