Commit message: fix: align Tracer mass with 30 kg specification and approximate inertias

File: HW/URDF/tracer/tracer_v1.urdf (robot description, URDF)
Before this commit: robot tracer_v1, 12 links, 11 joints
Links:
- link fl_castor_link: mass 1 -> 0.125
- link fl_wheel_link: mass 1 -> 0.125
- link fr_castor_link: mass 1 -> 0.125
- link fr_wheel_link: mass 1 -> 0.125
- link inertial_link: mass 132.3898489950015 -> 26
- link left_wheel_link: mass 6 -> 1.5
- link right_wheel_link: mass 6 -> 1.5
- link rl_castor_link: mass 1 -> 0.125
- link rl_wheel_link: mass 1 -> 0.125
- link rr_castor_link: mass 1 -> 0.125
- link rr_wheel_link: mass 1 -> 0.125

File: simulation/robot_description/tracer_sensor_rack_piper.urdf (robot description, URDF)
Before this commit: robot tracer_sensor_rack_piper, 86 links, 85 joints
Links:
- link fl_castor_link: mass 1 -> 0.125
- link fl_wheel_link: mass 1 -> 0.125
- link fr_castor_link: mass 1 -> 0.125
- link fr_wheel_link: mass 1 -> 0.125
- link inertial_link: mass 132.3898489950015 -> 26
- link left_wheel_link: mass 6 -> 1.5
- link right_wheel_link: mass 6 -> 1.5
- link rl_castor_link: mass 1 -> 0.125
- link rl_wheel_link: mass 1 -> 0.125
- link rr_castor_link: mass 1 -> 0.125
- link rr_wheel_link: mass 1 -> 0.125

File: simulation/robot_description/tracer_sensor_rack_piper_gazebo.urdf (robot description, URDF)
Before this commit: robot tracer_sensor_rack_piper, 85 links, 84 joints
Links:
- link fl_castor_link: mass 1 -> 0.125
- link fl_wheel_link: mass 1 -> 0.125
- link fr_castor_link: mass 1 -> 0.125
- link fr_wheel_link: mass 1 -> 0.125
- link inertial_link: mass 132.3898489950015 -> 26
- link left_wheel_link: mass 6 -> 1.5
- link right_wheel_link: mass 6 -> 1.5
- link rl_castor_link: mass 1 -> 0.125
- link rl_wheel_link: mass 1 -> 0.125
- link rr_castor_link: mass 1 -> 0.125
- link rr_wheel_link: mass 1 -> 0.125
