Commit message: Finalize single robot URDF and document simulation controls

File: simulation/robot_description/robocup.urdf (robot description, URDF)
Before this commit: robot tracer_sensor_rack_piper, 85 links, 84 joints
Links:
- added link wrist_camera_cad_link, mass 0.075; collision box size=0.089895801059 0.0249999577195 0.0256460003164; visual mesh filename=../../HW/URDF/wrist_camera_description/meshes/wrist_camera_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 scale=1 1 1
- added link wrist_camera_link
- added link wrist_camera_mount_link, mass 0.0150652381071; collision box size=0.06 0.013 0.0615; visual mesh filename=../../HW/URDF/wrist_camera_description/meshes/wrist_camera_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 scale=1 1 1
- added link wrist_camera_optical_frame
Joints:
- added joint piper_to_wrist_camera_mount: type fixed, parent piper_gripper_base, child wrist_camera_mount_link, origin xyz=1.4166402004356371e-05 2.7045737653415627e-05 0.00717003020070589 rpy=-1.5707995642548238 -1.2662970102272908e-05 1.6128249746224554
- added joint wrist_camera_body_frame: type fixed, parent wrist_camera_cad_link, child wrist_camera_link, origin xyz=0 0 0 rpy=-1.5707963267948966 -1.5707963267948966 0.0
- added joint wrist_camera_optical_joint: type fixed, parent wrist_camera_link, child wrist_camera_optical_frame, origin xyz=0 0 0 rpy=-1.5707963267948966 0 -1.5707963267948966
- added joint wrist_mount_to_camera: type fixed, parent wrist_camera_mount_link, child wrist_camera_cad_link, origin xyz=0 -0.02505 0.0665 rpy=1.5707963267948966 0 0

Commit message: Use the turned Piper arm pose as the assembled joint zero
Bake the original joint 1 angle of 1.6 rad into robocup.urdf, shift limits to preserve travel, and align shared manual controls. Keep the MuJoCo tutorial physical poses with offset coordinates and use current-model metadata in its export test. Preserve historical grasp data and document the required regeneration.

File: simulation/robot_description/robocup.urdf (robot description, URDF)
Before this commit: robot robocup, 89 links, 88 joints
Joints:
- joint piper_joint1: limit lower=-2.6179938 upper=2.6179938 effort=100 velocity=5 -> lower=-4.2179938 upper=1.0179938 effort=100 velocity=5; origin xyz=0 0 0.123 rpy=0 0 0 -> xyz=0 0 0.123 rpy=0 0 1.6

Commit message: Update rack geometry and Piper mounting pose from revised Fusion assembly

File: simulation/robot_description/robocup.urdf (robot description, URDF)
Before this commit: robot robocup, 89 links, 88 joints
Links:
- removed link cad_Manipulator_mount_1
- removed link cad_bracket_10
- removed link cad_bracket_12
- removed link cad_bracket_14
- removed link cad_bracket_15
- removed link cad_bracket_17
- removed link cad_bracket_9
- removed link cad_profiles_250mm_3
- removed link cad_profiles_250mm_4
- removed link cad_profiles_390mm_4
- removed link cad_profiles_500mm_1
- removed link cad_profiles_500mm_2
- removed link cad_profiles_500mm_3
- removed link cad_profiles_500mm_4
- added link cad_bracket_25
- added link cad_bracket_26
- added link cad_bracket_27
- added link cad_bracket_28
- added link cad_bracket_29
- added link cad_bracket_30
- added link cad_bracket_31
- added link cad_bracket_32
- added link cad_bracket_33
- added link cad_bracket_34
- added link cad_bracket_35
- added link cad_bracket_36
- added link cad_profiles_150mm_1
- added link cad_profiles_150mm_2
- added link cad_profiles_390mm_5
- added link cad_profiles_500mm_7
- added link cad_profiles_500mm_8
- added link cad_profiles_750mm_1
- added link cad_profiles_750mm_2
- link rack_base_link: mass 15.85407974 -> 15.6463681034; geometry collision box size=0.04 0.04 0.04; collision box size=0.04 0.04 0.04
Joints:
- removed joint cad_Manipulator_mount_1_joint
- removed joint cad_bracket_10_joint
- removed joint cad_bracket_12_joint
- removed joint cad_bracket_14_joint
- removed joint cad_bracket_15_joint
- removed joint cad_bracket_17_joint
- removed joint cad_bracket_9_joint
- removed joint cad_profiles_250mm_3_joint
- removed joint cad_profiles_250mm_4_joint
- removed joint cad_profiles_390mm_4_joint
- removed joint cad_profiles_500mm_1_joint
- removed joint cad_profiles_500mm_2_joint
- removed joint cad_profiles_500mm_3_joint
- removed joint cad_profiles_500mm_4_joint
- added joint cad_bracket_25_joint: type fixed, parent rack_base_link, child cad_bracket_25, origin xyz=-0.16 -0.222980453529 0.235659132024 rpy=1.57079632679 6.12323399574e-17 1.57079632679
- added joint cad_bracket_26_joint: type fixed, parent rack_base_link, child cad_bracket_26, origin xyz=-0.16 0.206669546471 0.235659132024 rpy=1.57079632679 6.12323399574e-17 1.57079632679
- added joint cad_bracket_27_joint: type fixed, parent rack_base_link, child cad_bracket_27, origin xyz=0.0443408679762 0.206669546471 0.29 rpy=6.12323399574e-17 6.12323399574e-17 1.57079632679
- added joint cad_bracket_28_joint: type fixed, parent rack_base_link, child cad_bracket_28, origin xyz=-0.0243408679762 0.222980453529 0.29 rpy=-6.12323399574e-17 -6.12323399574e-17 -1.57079632679
- added joint cad_bracket_29_joint: type fixed, parent rack_base_link, child cad_bracket_29, origin xyz=0.0443408679762 -0.222980453529 0.29 rpy=6.12323399574e-17 6.12323399574e-17 1.57079632679
- added joint cad_bracket_30_joint: type fixed, parent rack_base_link, child cad_bracket_30, origin xyz=-0.0243408679762 -0.206669546471 0.29 rpy=-6.12323399574e-17 -6.12323399574e-17 -1.57079632679
- added joint cad_bracket_31_joint: type fixed, parent rack_base_link, child cad_bracket_31, origin xyz=0.00166954647057 0.195 0.735659132024 rpy=1.57079632679 -5.55111512313e-16 -5.55111512313e-16
- added joint cad_bracket_32_joint: type fixed, parent rack_base_link, child cad_bracket_32, origin xyz=0.00166954647057 -0.180659132024 0.75 rpy=-3.14159265359 2.62999016384e-32 -1.11022302463e-15
- added joint cad_bracket_33_joint: type fixed, parent rack_base_link, child cad_bracket_33, origin xyz=-0.145659132024 -0.055 0.761669546471 rpy=0 -1.57079632679 1.57079632679
- added joint cad_bracket_34_joint: type fixed, parent rack_base_link, child cad_bracket_34, origin xyz=-0.16 0.0693408679762 0.762019546471 rpy=0 -1.57079632679 3.14159265359
- added joint cad_bracket_35_joint: type fixed, parent rack_base_link, child cad_bracket_35, origin xyz=-0.01 0.0693408679762 0.777980453529 rpy=0 1.57079632679 3.14159265359
- added joint cad_bracket_36_joint: type fixed, parent rack_base_link, child cad_bracket_36, origin xyz=-0.01 -0.0693408679762 0.761669546471 rpy=0 -1.57079632679 -2.66113378704e-16
- added joint cad_profiles_150mm_1_joint: type fixed, parent rack_base_link, child cad_profiles_150mm_1, origin xyz=-0.11 -0.00771129415511 0.797772226096 rpy=-4.65274880733e-47 8.62816615085e-32 -1.57079632679
- added joint cad_profiles_150mm_2_joint: type fixed, parent rack_base_link, child cad_profiles_150mm_2, origin xyz=-0.11 0.0622887058449 0.797772226096 rpy=-3.69482993523e-47 8.62816615085e-32 -1.57079632679
- added joint cad_profiles_390mm_5_joint: type fixed, parent rack_base_link, child cad_profiles_390mm_5, origin xyz=-0.0172887058449 0.095 0.797772226096 rpy=7.39557098645e-32 -4.1681652034e-32 -5.55111512313e-16
- added joint cad_profiles_500mm_7_joint: type fixed, parent rack_base_link, child cad_profiles_500mm_7, origin xyz=-0.0172887058449 -0.242772226096 0.69 rpy=1.57079632679 1.63688800411e-32 0
- added joint cad_profiles_500mm_8_joint: type fixed, parent rack_base_link, child cad_profiles_500mm_8, origin xyz=-0.0172887058449 0.187227773904 0.69 rpy=1.57079632679 -4.1681652034e-32 0
- added joint cad_profiles_750mm_1_joint: type fixed, parent rack_base_link, child cad_profiles_750mm_1, origin xyz=-0.207288705845 -0.242772226096 0.69 rpy=1.57079632679 3.59611246825e-46 0
- added joint cad_profiles_750mm_2_joint: type fixed, parent rack_base_link, child cad_profiles_750mm_2, origin xyz=-0.207288705845 0.187227773904 0.69 rpy=1.57079632679 -7.02652359554e-46 0
- joint cad_bracket_11_joint: origin xyz=-0.145659132 -0.2229804535 0.29 rpy=6.12323399574e-17 6.12323399574e-17 1.57079632679 -> xyz=-0.145659132024 -0.222980453529 0.29 rpy=6.12323399574e-17 6.12323399574e-17 1.57079632679
- joint cad_bracket_13_joint: origin xyz=-0.145659132 0.2066695465 0.29 rpy=2.8187954982e-16 6.12323399574e-17 1.57079632679 -> xyz=-0.145659132024 0.206669546471 0.29 rpy=2.8187954982e-16 6.12323399574e-17 1.57079632679
- joint cad_bracket_16_joint: origin xyz=-0.1883304535 0.195 0.735659132 rpy=1.57079632679 -3.88578058619e-16 -3.88578058619e-16 -> xyz=-0.188330453529 0.195 0.735659132024 rpy=1.57079632679 -3.88578058619e-16 -3.88578058619e-16
- joint cad_bracket_18_joint: origin xyz=-0.1883304535 -0.180659132 0.75 rpy=-3.14159265359 -1.14802924234e-29 -3.2457918806e-45 -> xyz=-0.188330453529 -0.180659132024 0.75 rpy=-3.14159265359 -1.14802924234e-29 -3.2457918806e-45
- joint cad_bracket_1_joint: origin xyz=0.08 0.180659132 0.2778054535 rpy=0 1.57079632679 -1.27675647832e-15 -> xyz=0.08 0.180659132024 0.277805453529 rpy=0 1.57079632679 -1.27675647832e-15
- joint cad_bracket_21_joint: origin xyz=-0.1883304535 0.110659132 0.79 rpy=1.26957301934e-29 -1.47911419727e-31 -1.87784347738e-60 -> xyz=-0.188330453529 0.110659132024 0.79 rpy=1.26957301934e-29 -1.47911419727e-31 -1.87784347738e-60
- joint cad_bracket_22_joint: origin xyz=-0.1883304535 -0.125 0.804340868 rpy=-1.57079632679 3.22939933075e-29 -3.22939933075e-29 -> xyz=-0.188330453529 -0.125 0.804340867976 rpy=-1.57079632679 3.22939933075e-29 -3.22939933075e-29
- joint cad_bracket_23_joint: origin xyz=-0.1883304535 -0.110659132 1.25 rpy=-3.14159265359 2.81252462387e-42 -7.03230078465e-71 -> xyz=-0.188330453529 -0.110659132024 1.25 rpy=-3.14159265359 2.81252462387e-42 -7.03230078465e-71
- joint cad_bracket_24_joint: origin xyz=-0.1883304535 0.125 1.235659132 rpy=1.57079632679 2.81252462387e-42 0 -> xyz=-0.188330453529 0.125 1.23565913202 rpy=1.57079632679 2.81252462387e-42 0
- joint cad_bracket_2_joint: origin xyz=0.02565913202 0.195 0.2779804535 rpy=0 1.57079632679 -1.57079632679 -> xyz=0.0256591320238 0.195 0.277980453529 rpy=0 1.57079632679 -1.57079632679
- joint cad_bracket_3_joint: origin xyz=-0.02565913202 0.195 0.2616695465 rpy=0 -1.57079632679 1.57079632679 -> xyz=-0.0256591320238 0.195 0.261669546471 rpy=0 -1.57079632679 1.57079632679
- joint cad_bracket_4_joint: origin xyz=-0.08 0.180659132 0.2616695465 rpy=0 -1.57079632679 3.53572290739e-16 -> xyz=-0.08 0.180659132024 0.261669546471 rpy=0 -1.57079632679 3.53572290739e-16
- joint cad_bracket_5_joint: origin xyz=0.08 -0.180659132 0.2616695465 rpy=0 -1.57079632679 3.14159265359 -> xyz=0.08 -0.180659132024 0.261669546471 rpy=0 -1.57079632679 3.14159265359
- joint cad_bracket_6_joint: origin xyz=0.02565913202 -0.195 0.2616695465 rpy=0 -1.57079632679 -1.57079632679 -> xyz=0.0256591320238 -0.195 0.261669546471 rpy=0 -1.57079632679 -1.57079632679
- joint cad_bracket_7_joint: origin xyz=-0.04 -0.180659132 0.2616695465 rpy=0 -1.57079632679 3.14159265359 -> xyz=-0.04 -0.180659132024 0.261669546471 rpy=0 -1.57079632679 3.14159265359
- joint cad_bracket_8_joint: origin xyz=-0.08 -0.180659132 0.2779804535 rpy=0 1.57079632679 -3.14159265359 -> xyz=-0.08 -0.180659132024 0.277980453529 rpy=0 1.57079632679 -3.14159265359
- joint cad_profiles_250mm_1_joint: origin xyz=0.1527112942 0.1872277739 0.19 rpy=1.57079632679 -0 0 -> xyz=0.152711294155 0.187227773904 0.19 rpy=1.57079632679 -0 0
- joint cad_profiles_250mm_2_joint: origin xyz=0.1527112942 -0.2427722261 0.19 rpy=1.57079632679 -0 0 -> xyz=0.152711294155 -0.242772226096 0.19 rpy=1.57079632679 -0 0
- joint cad_profiles_250mm_5_joint: origin xyz=-0.2072887058 0.025 1.297772226 rpy=-1.25108409187e-29 2.81252462387e-42 -3.51870481493e-71 -> xyz=-0.207288705845 0.025 1.2977722261 rpy=-1.25108409187e-29 2.81252462387e-42 -3.51870481493e-71
- joint cad_profiles_320mm_1_joint: origin xyz=-0.06 -0.2422887058 0.0477722261 rpy=-3.41377878841e-17 6.07153216592e-18 1.57079632679 -> xyz=-0.06 -0.242288705845 0.0477722260964 rpy=-3.41377878841e-17 6.07153216592e-18 1.57079632679
- joint cad_profiles_320mm_2_joint: origin xyz=-0.06 0.1877112942 0.0477722261 rpy=0 -0 1.57079632679 -> xyz=-0.06 0.187711294155 0.0477722260964 rpy=0 -0 1.57079632679
- joint cad_profiles_320mm_3_joint: origin xyz=-0.06 -0.2422887058 0.2977722261 rpy=6.12323399574e-17 6.12323399574e-17 1.57079632679 -> xyz=-0.06 -0.242288705845 0.297772226096 rpy=6.12323399574e-17 6.12323399574e-17 1.57079632679
- joint cad_profiles_320mm_4_joint: origin xyz=-0.06 0.1877112942 0.2977722261 rpy=6.12323399574e-17 6.12323399574e-17 1.57079632679 -> xyz=-0.06 0.187711294155 0.297772226096 rpy=6.12323399574e-17 6.12323399574e-17 1.57079632679
- joint cad_profiles_390mm_1_joint: origin xyz=0.03271129416 0.095 0.2977722261 rpy=1.10933564797e-31 1.41635147517e-46 -1.27675647832e-15 -> xyz=0.0327112941551 0.095 0.297772226096 rpy=1.10933564797e-31 1.41635147517e-46 -1.27675647832e-15
- joint cad_profiles_390mm_2_joint: origin xyz=-0.08728870584 0.095 0.2977722261 rpy=2.4612511597e-62 -1.10933564797e-31 1.36517682503e-93 -> xyz=-0.0872887058449 0.095 0.297772226096 rpy=2.4612511597e-62 -1.10933564797e-31 1.36517682503e-93
- joint cad_profiles_390mm_3_joint: origin xyz=-0.2072887058 0.095 0.7977722261 rpy=8.62816615085e-32 -1.10933564797e-31 -3.88578058619e-16 -> xyz=-0.207288705845 0.095 0.797772226096 rpy=8.62816615085e-32 -1.10933564797e-31 -3.88578058619e-16
- joint cad_profiles_470mm_1_joint: origin xyz=0.1527112942 0.135 0.0477722261 rpy=0 -0 0 -> xyz=0.152711294155 0.135 0.0477722260964 rpy=0 -0 0
- joint cad_profiles_470mm_2_joint: origin xyz=-0.2072887058 0.135 0.0477722261 rpy=0 -0 1.10933564797e-31 -> xyz=-0.207288705845 0.135 0.0477722260964 rpy=0 -0 1.10933564797e-31
- joint cad_profiles_500mm_5_joint: origin xyz=-0.2072887058 -0.1727722261 1.19 rpy=1.57079632679 2.81252462387e-42 -3.22939933075e-29 -> xyz=-0.207288705845 -0.172772226096 1.19 rpy=1.57079632679 2.81252462387e-42 -3.22939933075e-29
- joint cad_profiles_500mm_6_joint: origin xyz=-0.2072887058 0.1172277739 1.19 rpy=1.57079632679 -1.47911419727e-31 -1.82362454574e-29 -> xyz=-0.207288705845 0.117227773904 1.19 rpy=1.57079632679 -1.47911419727e-31 -1.82362454574e-29
- joint rack_to_piper_base: origin xyz=0 0 0.0038 rpy=0 0 0 -> xyz=-0.0195 -2.00728322852e-15 0.79 rpy=0 0 0; parent cad_Manipulator_mount_1 -> rack_base_link
