Commit message: Apply physical G2 calibration against Mid-360S to the calibrated URDF
Static multi-pose estimate of base_link <- laser_frame on the real robot
(2026-10-10): x=24.248 mm, y=9.159 mm, yaw=2.8367 deg; z/roll/pitch kept
from CAD. CAD yaw was 8.81 deg. 6 train / 2 held-out poses; held-out
G2-to-Mid-360S wall distance median 7.0/6.7 mm (CAD 42/70 mm).

- HW/calibration/base_2dlidar: record, per-pose results, solver output,
  collection/solver tools. Raw bags stay on the Jetson (SHA-256 listed).
- integrate_calibration.py reads the physical record instead of the
  Gazebo 20261005_base_2dlidar record (kept as history).
- Regenerated robocup.calibrated.urdf: only laser_frame_joint changes
  semantically. The integrated bundle is regenerated too, which also
  brings results/base_head.json in line with the 15 deg mount already
  in the runtime URDF.

Co-Authored-By: Claude Opus 5.5 <noreply@anthropic.com>

File: SW/simulation/calibration/records/integrated_calibration/application/base_head.urdf (robot description, URDF)
Before this commit: robot robocup, 94 links, 93 joints
Links:
- link rack_base_link: mass 15.6463681034 -> 15.6921304573; geometry collision box size=0.04 0.04 0.04; collision box size=0.04 0.04 0.04
Joints:
- joint cad_D435f_Solid_v1_1_joint: origin xyz=-0.12495 -2.611244554e-15 1.27 rpy=1.57079632679 1.25108409187e-29 1.57079632679 -> xyz=-0.120666319792 0.00125 1.26068901712 rpy=1.83259571459 1.2669865157e-12 1.57079632679
- joint camera_link_joint: origin xyz=-0.12722342972197517 -0.001716274462443348 1.2689368986951095 rpy=0.0037066991262989625 -0.0043934350517067511 0.0014976471610455334 -> xyz=-0.1231374351388152 -0.00046627446244331891 1.2602505470202274 rpy=0.0041075243142279123 0.25740565260292736 0.0015486552345582768
- joint laser_frame_joint: origin xyz=-5.1389834908760446e-05 0.00052051635559500814 0 rpy=0 0 0.15437059215843318 -> xyz=0.024073172308992453 0.0091594372740952668 0 rpy=0 0 0.049509674634016343
- joint livox_frame_joint: origin xyz=3.773355003483525e-05 0.00015620113972823895 -0.00024318079626794997 rpy=3.1415281256409191 2.0508080655012861e-05 -2.7091518517208257e-05 -> xyz=3.773355003483525e-05 0.00015620113972823895 -0.00024318079626794997 rpy=3.1415281256409195 2.0508080655234906e-05 -2.7091518517184195e-05

File: SW/simulation/calibration/records/integrated_calibration/application/base_lidar.urdf (robot description, URDF)
Before this commit: robot robocup, 94 links, 93 joints
Links:
- link rack_base_link: mass 15.6463681034 -> 15.6921304573; geometry collision box size=0.04 0.04 0.04; collision box size=0.04 0.04 0.04
Joints:
- joint cad_D435f_Solid_v1_1_joint: origin xyz=-0.12495 -2.611244554e-15 1.27 rpy=1.57079632679 1.25108409187e-29 1.57079632679 -> xyz=-0.120666319792 0.00125 1.26068901712 rpy=1.83259571459 1.2669865157e-12 1.57079632679
- joint camera_link_joint: origin xyz=-0.12495 -2.611244554e-15 1.27 rpy=0 0 0 -> xyz=-0.120666319792 0.00125 1.26068901712 rpy=5.29217496717e-18 0.261799387799 -1.34215948492e-17
- joint laser_frame_joint: origin xyz=-5.1389834908760446e-05 0.00052051635559500814 0 rpy=0 0 0.15437059215843318 -> xyz=0.024073172308992453 0.0091594372740952668 0 rpy=0 0 0.049509674634016343

File: SW/simulation/calibration/records/integrated_calibration/application/base_mid360.urdf (robot description, URDF)
Before this commit: robot robocup, 94 links, 93 joints
Links:
- link rack_base_link: mass 15.6463681034 -> 15.6921304573; geometry collision box size=0.04 0.04 0.04; collision box size=0.04 0.04 0.04
Joints:
- joint cad_D435f_Solid_v1_1_joint: origin xyz=-0.12495 -2.611244554e-15 1.27 rpy=1.57079632679 1.25108409187e-29 1.57079632679 -> xyz=-0.120666319792 0.00125 1.26068901712 rpy=1.83259571459 1.2669865157e-12 1.57079632679
- joint camera_link_joint: origin xyz=-0.12495 -2.611244554e-15 1.27 rpy=0 0 0 -> xyz=-0.120666319792 0.00125 1.26068901712 rpy=5.29217496717e-18 0.261799387799 -1.34215948492e-17
- joint laser_frame_joint: origin xyz=-5.1389834908760446e-05 0.00052051635559500814 0 rpy=0 0 0.15437059215843318 -> xyz=0.024073172308992453 0.0091594372740952668 0 rpy=0 0 0.049509674634016343
- joint livox_frame_joint: origin xyz=3.773355003483525e-05 0.00015620113972823895 -0.00024318079626794997 rpy=3.1415281256409191 2.0508080655012861e-05 -2.7091518517208257e-05 -> xyz=3.773355003483525e-05 0.00015620113972823895 -0.00024318079626794997 rpy=3.1415281256409195 2.0508080655234906e-05 -2.7091518517184195e-05

File: SW/simulation/calibration/records/integrated_calibration/application/base_piper.urdf (robot description, URDF)
Before this commit: robot robocup, 94 links, 93 joints
Links:
- link rack_base_link: mass 15.6463681034 -> 15.6921304573; geometry collision box size=0.04 0.04 0.04; collision box size=0.04 0.04 0.04
Joints:
- joint cad_D435f_Solid_v1_1_joint: origin xyz=-0.12495 -2.611244554e-15 1.27 rpy=1.57079632679 1.25108409187e-29 1.57079632679 -> xyz=-0.120666319792 0.00125 1.26068901712 rpy=1.83259571459 1.2669865157e-12 1.57079632679
- joint camera_link_joint: origin xyz=-0.12495 -2.611244554e-15 1.27 rpy=0 0 0 -> xyz=-0.120666319792 0.00125 1.26068901712 rpy=5.29217496717e-18 0.261799387799 -1.34215948492e-17
- joint laser_frame_joint: origin xyz=-5.1389834908760446e-05 0.00052051635559500814 0 rpy=0 0 0.15437059215843318 -> xyz=0.024073172308992453 0.0091594372740952668 0 rpy=0 0 0.049509674634016343
- joint livox_frame_joint: origin xyz=3.773355003483525e-05 0.00015620113972823895 -0.00024318079626794997 rpy=3.1415281256409191 2.0508080655012861e-05 -2.7091518517208257e-05 -> xyz=3.773355003483525e-05 0.00015620113972823895 -0.00024318079626794997 rpy=3.1415281256409195 2.0508080655234906e-05 -2.7091518517184195e-05

File: SW/simulation/calibration/records/integrated_calibration/application/flange_wrist.urdf (robot description, URDF)
Before this commit: robot robocup, 94 links, 93 joints
Links:
- link rack_base_link: mass 15.6463681034 -> 15.6921304573; geometry collision box size=0.04 0.04 0.04; collision box size=0.04 0.04 0.04
Joints:
- joint cad_D435f_Solid_v1_1_joint: origin xyz=-0.12495 -2.611244554e-15 1.27 rpy=1.57079632679 1.25108409187e-29 1.57079632679 -> xyz=-0.120666319792 0.00125 1.26068901712 rpy=1.83259571459 1.2669865157e-12 1.57079632679
- joint camera_link_joint: origin xyz=-0.12722342972197517 -0.001716274462443348 1.2689368986951095 rpy=0.0037066991262989625 -0.0043934350517067511 0.0014976471610455334 -> xyz=-0.1231374351388152 -0.00046627446244331891 1.2602505470202274 rpy=0.0041075243142279123 0.25740565260292736 0.0015486552345582768
- joint laser_frame_joint: origin xyz=-5.1389834908760446e-05 0.00052051635559500814 0 rpy=0 0 0.15437059215843318 -> xyz=0.024073172308992453 0.0091594372740952668 0 rpy=0 0 0.049509674634016343
- joint livox_frame_joint: origin xyz=3.773355003483525e-05 0.00015620113972823895 -0.00024318079626794997 rpy=3.1415281256409191 2.0508080655012861e-05 -2.7091518517208257e-05 -> xyz=3.773355003483525e-05 0.00015620113972823895 -0.00024318079626794997 rpy=3.1415281256409195 2.0508080655234906e-05 -2.7091518517184195e-05
- joint piper_to_wrist_camera_mount: origin xyz=0.00021057778731321184 0.00081284728291651563 0.0072422552841638725 rpy=-1.5721318918257796 -0.0019379665882315322 1.6152889735146658 -> xyz=0.00021057778731321808 0.00081284728291651596 0.0072422552841638725 rpy=-1.5721318918257798 -0.0019379665882315322 1.6152889735146665

File: SW/simulation/robot_description/robocup.calibrated.urdf (robot description, URDF)
Before this commit: robot robocup, 95 links, 94 joints
Joints:
- joint camera_link_joint: origin xyz=-0.123137435139 -0.000466274462443 1.26025054702 rpy=0.00410752431423 0.257405652603 0.00154865523456 -> xyz=-0.1231374351388152 -0.00046627446244331891 1.2602505470202274 rpy=0.0041075243142279123 0.25740565260292736 0.0015486552345582768
- joint laser_frame_joint: origin xyz=-5.1389834908760446e-05 0.00052051635559500814 0 rpy=0 0 0.15437059215843318 -> xyz=0.024073172308992453 0.0091594372740952668 0 rpy=0 0 0.049509674634016343
- joint livox_frame_joint: origin xyz=3.773355003483525e-05 0.00015620113972823895 -0.00024318079626794997 rpy=3.1415281256409191 2.0508080655012861e-05 -2.7091518517208257e-05 -> xyz=3.773355003483525e-05 0.00015620113972823895 -0.00024318079626794997 rpy=3.1415281256409195 2.0508080655234906e-05 -2.7091518517184195e-05
- joint piper_to_wrist_camera_mount: origin xyz=0.00021057778731321184 0.00081284728291651563 0.0072422552841638725 rpy=-1.5721318918257796 -0.0019379665882315322 1.6152889735146658 -> xyz=0.00021057778731321808 0.00081284728291651596 0.0072422552841638725 rpy=-1.5721318918257798 -0.0019379665882315322 1.6152889735146665

Commit message: Calibrate G2 and Mid-360S against base_link; correct Tracer odometry
G2 (base_link <- laser_frame), motion geometry from the team's stop-and-go
spin/straight bags: x=3.05 mm, y=6.76 mm, yaw=1.2176 deg (CAD 8.81 deg).
CW/CCW rotation centres agree within 2.7 mm, forward/reverse yaw within
0.02 deg. Odometry magnitudes are not used.

Mid-360S (base_link <- livox_frame): real floor plane gives pitch 2.906 deg
/ roll 0.12 deg (matches the internal IMU) and z; x/y/yaw from the G2 chain
after re-fitting G2 to the tilt-corrected Mid-360S map (held-out wall
distance median 6.8 mm, 6-DoF diagnostic pitch now 0.02 deg). Result
(-158.0, 0.1, 1188.5) mm, rpy (-179.88, 2.906, -1.607) deg.

The previous G2 value relative to an untilted CAD Mid-360S is kept under
base_2dlidar/vs_mid360 as history; its floor diagnostics were wrong.

Tracer odometry: v = 1.112 v_rep, w = 1.319 w_rep + 0.00378 rad/s while
moving. Applied on the Jetson in a local tracer_ros2 branch; the patch is
recorded under HW/calibration/tracer_odom.

robocup.calibrated.urdf: only laser_frame_joint and livox_frame_joint change.

Co-Authored-By: Claude Opus 5.5 <noreply@anthropic.com>

File: SW/simulation/calibration/records/integrated_calibration/application/base_head.urdf (robot description, URDF)
Before this commit: robot robocup, 94 links, 93 joints
Joints:
- joint laser_frame_joint: origin xyz=0.024073172308992453 0.0091594372740952668 0 rpy=0 0 0.049509674634016343 -> xyz=0.0028733029026841292 0.0067586514684851492 0 rpy=0 0 0.021251994651100784
- joint livox_frame_joint: origin xyz=3.773355003483525e-05 0.00015620113972823895 -0.00024318079626794997 rpy=3.1415281256409195 2.0508080655234906e-05 -2.7091518517184195e-05 -> xyz=0.022032700644211894 5.7685849495536964e-05 -0.010564391472523305 rpy=-3.1395053590522144 0.050714699081705339 -0.028042824854912916

File: SW/simulation/calibration/records/integrated_calibration/application/base_lidar.urdf (robot description, URDF)
Before this commit: robot robocup, 94 links, 93 joints
Joints:
- joint laser_frame_joint: origin xyz=0.024073172308992453 0.0091594372740952668 0 rpy=0 0 0.049509674634016343 -> xyz=0.0028733029026841292 0.0067586514684851492 0 rpy=0 0 0.021251994651100784

File: SW/simulation/calibration/records/integrated_calibration/application/base_mid360.urdf (robot description, URDF)
Before this commit: robot robocup, 94 links, 93 joints
Joints:
- joint laser_frame_joint: origin xyz=0.024073172308992453 0.0091594372740952668 0 rpy=0 0 0.049509674634016343 -> xyz=0.0028733029026841292 0.0067586514684851492 0 rpy=0 0 0.021251994651100784
- joint livox_frame_joint: origin xyz=3.773355003483525e-05 0.00015620113972823895 -0.00024318079626794997 rpy=3.1415281256409195 2.0508080655234906e-05 -2.7091518517184195e-05 -> xyz=0.022032700644211894 5.7685849495536964e-05 -0.010564391472523305 rpy=-3.1395053590522144 0.050714699081705339 -0.028042824854912916

File: SW/simulation/calibration/records/integrated_calibration/application/base_piper.urdf (robot description, URDF)
Before this commit: robot robocup, 94 links, 93 joints
Joints:
- joint laser_frame_joint: origin xyz=0.024073172308992453 0.0091594372740952668 0 rpy=0 0 0.049509674634016343 -> xyz=0.0028733029026841292 0.0067586514684851492 0 rpy=0 0 0.021251994651100784
- joint livox_frame_joint: origin xyz=3.773355003483525e-05 0.00015620113972823895 -0.00024318079626794997 rpy=3.1415281256409195 2.0508080655234906e-05 -2.7091518517184195e-05 -> xyz=0.022032700644211894 5.7685849495536964e-05 -0.010564391472523305 rpy=-3.1395053590522144 0.050714699081705339 -0.028042824854912916

File: SW/simulation/calibration/records/integrated_calibration/application/flange_wrist.urdf (robot description, URDF)
Before this commit: robot robocup, 94 links, 93 joints
Joints:
- joint laser_frame_joint: origin xyz=0.024073172308992453 0.0091594372740952668 0 rpy=0 0 0.049509674634016343 -> xyz=0.0028733029026841292 0.0067586514684851492 0 rpy=0 0 0.021251994651100784
- joint livox_frame_joint: origin xyz=3.773355003483525e-05 0.00015620113972823895 -0.00024318079626794997 rpy=3.1415281256409195 2.0508080655234906e-05 -2.7091518517184195e-05 -> xyz=0.022032700644211894 5.7685849495536964e-05 -0.010564391472523305 rpy=-3.1395053590522144 0.050714699081705339 -0.028042824854912916

File: SW/simulation/robot_description/robocup.calibrated.urdf (robot description, URDF)
Before this commit: robot robocup, 95 links, 94 joints
Joints:
- joint laser_frame_joint: origin xyz=0.024073172308992453 0.0091594372740952668 0 rpy=0 0 0.049509674634016343 -> xyz=0.0028733029026841292 0.0067586514684851492 0 rpy=0 0 0.021251994651100784
- joint livox_frame_joint: origin xyz=3.773355003483525e-05 0.00015620113972823895 -0.00024318079626794997 rpy=3.1415281256409195 2.0508080655234906e-05 -2.7091518517184195e-05 -> xyz=0.022032700644211894 5.7685849495536964e-05 -0.010564391472523305 rpy=-3.1395053590522144 0.050714699081705339 -0.028042824854912916

Commit message: Address cross-review: hold-out separation, floor-consistent z, offset odom model
Mid-360S: floor tilt from pose01-03 only (hold-out pose04/08 untouched);
z from the mean sensor-to-floor distance; hold-out evaluated with the
deployed transforms (median 6.6 mm, p90 16.4 mm vs 6.9 / 18.8 mm without
tilt). Result (-158.8, 0.8, 1190.6) mm, rpy (-179.92, 2.847, -1.609) deg.
Absolute z is not independently verified (tape -22 mm).

Odometry: the firmware speeds are short by a roughly constant amount; an
offset model (v +0.00443 m/s, w +0.0523 rad/s above 0.04 rad/s) beats the
scale model in cross-validation between two sessions (rotation 1.5-1.7
deg vs 3-6 deg per segment). Driver commit ad78440 with typed launch
parameters; the patch file covers both driver commits.

integrate_calibration.py: provisional numeric quality limits and a check
that the Mid-360S record was derived from the current G2 record.
Tools take paths as arguments; added check_poses.py, odom_validate.py,
odom_model_cv.py.

Co-Authored-By: Claude Opus 5.5 <noreply@anthropic.com>

File: SW/simulation/calibration/records/integrated_calibration/application/base_head.urdf (robot description, URDF)
Before this commit: robot robocup, 94 links, 93 joints
Joints:
- joint livox_frame_joint: origin xyz=0.022032700644211894 5.7685849495536964e-05 -0.010564391472523305 rpy=-3.1395053590522144 0.050714699081705339 -0.028042824854912916 -> xyz=0.021225211019230833 0.00082800074531052279 -0.0085105672975474 rpy=-3.1402789720886934 0.049694486354240341 -0.028090124176819987

File: SW/simulation/calibration/records/integrated_calibration/application/base_mid360.urdf (robot description, URDF)
Before this commit: robot robocup, 94 links, 93 joints
Joints:
- joint livox_frame_joint: origin xyz=0.022032700644211894 5.7685849495536964e-05 -0.010564391472523305 rpy=-3.1395053590522144 0.050714699081705339 -0.028042824854912916 -> xyz=0.021225211019230833 0.00082800074531052279 -0.0085105672975474 rpy=-3.1402789720886934 0.049694486354240341 -0.028090124176819987

File: SW/simulation/calibration/records/integrated_calibration/application/base_piper.urdf (robot description, URDF)
Before this commit: robot robocup, 94 links, 93 joints
Joints:
- joint livox_frame_joint: origin xyz=0.022032700644211894 5.7685849495536964e-05 -0.010564391472523305 rpy=-3.1395053590522144 0.050714699081705339 -0.028042824854912916 -> xyz=0.021225211019230833 0.00082800074531052279 -0.0085105672975474 rpy=-3.1402789720886934 0.049694486354240341 -0.028090124176819987

File: SW/simulation/calibration/records/integrated_calibration/application/flange_wrist.urdf (robot description, URDF)
Before this commit: robot robocup, 94 links, 93 joints
Joints:
- joint livox_frame_joint: origin xyz=0.022032700644211894 5.7685849495536964e-05 -0.010564391472523305 rpy=-3.1395053590522144 0.050714699081705339 -0.028042824854912916 -> xyz=0.021225211019230833 0.00082800074531052279 -0.0085105672975474 rpy=-3.1402789720886934 0.049694486354240341 -0.028090124176819987

File: SW/simulation/robot_description/robocup.calibrated.urdf (robot description, URDF)
Before this commit: robot robocup, 95 links, 94 joints
Joints:
- joint livox_frame_joint: origin xyz=0.022032700644211894 5.7685849495536964e-05 -0.010564391472523305 rpy=-3.1395053590522144 0.050714699081705339 -0.028042824854912916 -> xyz=0.021225211019230833 0.00082800074531052279 -0.0085105672975474 rpy=-3.1402789720886934 0.049694486354240341 -0.028090124176819987
