Commit message: Integrate Head hand-eye, Wrist, arm mount and nominal gripper TCP
Collect 25 training and 10 held-out Head–PiPER observations; select the arm Head route and preserve the earlier plane estimate. Apply sensor estimates and explicit URDF mount/TCP references in a portable runtime. Record the 9.871 mm Head route difference and remaining independent physical measurements.

File: SW/simulation/robot_description/robocup.calibrated.urdf (robot description, URDF)
Before this commit: robot robocup, 94 links, 93 joints
Links:
- added link tcp
Joints:
- added joint calibrated_tcp_joint: type fixed, parent piper_link6, child tcp, origin xyz=0.0 0.0 0.14250000000000002 rpy=0.0 0.0 0.0
- joint camera_link_joint: origin xyz=-0.12495 -2.611244554e-15 1.27 rpy=0 0 0 -> xyz=-0.12722342972197517 -0.001716274462443348 1.2689368986951095 rpy=0.0037066991262989625 -0.0043934350517067511 0.0014976471610455334
- joint piper_to_wrist_camera_mount: origin xyz=1.4166402004356371e-05 2.7045737653415627e-05 0.00717003020070589 rpy=-1.5707995642548238 -1.2662970102272908e-05 1.6128249746224554 -> xyz=0.00021057778731321184 0.00081284728291651563 0.0072422552841638725 rpy=-1.5721318918257796 -0.0019379665882315322 1.6152889735146658
- joint rack_to_piper_base: origin xyz=-0.0195 -2.00728322852e-15 0.79 rpy=0 0 0 -> xyz=-0.0195 -2.0072832285199999e-15 0.79000000000000004 rpy=0 0 0

Commit message: Complete simulated TCP pivot calibration and integrate runtime

File: SW/simulation/robot_description/robocup.calibrated.urdf (robot description, URDF)
Before this commit: robot robocup, 95 links, 94 joints
Joints:
- joint calibrated_tcp_joint: origin xyz=0.0 0.0 0.14250000000000002 rpy=0.0 0.0 0.0 -> xyz=3.1410601675219113e-09 -6.041407414281427e-10 0.14250000226360077 rpy=0.0 0.0 0.0

Commit message: Use selected Fusion 15 degree head camera mount as the default robot model

File: SW/simulation/robot_description/robocup.calibrated.urdf (robot description, URDF)
Before this commit: robot robocup, 95 links, 94 joints
Links:
- link rack_base_link: mass 15.6463681034 -> 15.6921304573; geometry collision box size=0.04 0.04 0.04; collision box size=0.04 0.04 0.04
Joints:
- joint cad_D435f_Solid_v1_1_joint: origin xyz=-0.12495 -2.611244554e-15 1.27 rpy=1.57079632679 1.25108409187e-29 1.57079632679 -> xyz=-0.120666319792 0.00125 1.26068901712 rpy=1.83259571459 1.2669865157e-12 1.57079632679
- joint camera_link_joint: origin xyz=-0.12722342972197517 -0.001716274462443348 1.2689368986951095 rpy=0.0037066991262989625 -0.0043934350517067511 0.0014976471610455334 -> xyz=-0.123137435139 -0.000466274462443 1.26025054702 rpy=0.00410752431423 0.257405652603 0.00154865523456

File: SW/simulation/robot_description/robocup.urdf (robot description, URDF)
Before this commit: robot robocup, 94 links, 93 joints
Links:
- link rack_base_link: mass 15.6463681034 -> 15.6921304573; geometry collision box size=0.04 0.04 0.04; collision box size=0.04 0.04 0.04
Joints:
- joint cad_D435f_Solid_v1_1_joint: origin xyz=-0.12495 -2.611244554e-15 1.27 rpy=1.57079632679 1.25108409187e-29 1.57079632679 -> xyz=-0.120666319792 0.00125 1.26068901712 rpy=1.83259571459 1.2669865157e-12 1.57079632679
- joint camera_link_joint: origin xyz=-0.12495 -2.611244554e-15 1.27 rpy=0 0 0 -> xyz=-0.120666319792 0.00125 1.26068901712 rpy=5.29217496717e-18 0.261799387799 -1.34215948492e-17

Commit message: Apply accepted koide3 Head–Mid360 calibration and Jetson sensor TF
Preserve the 2026-10-12 four-bag result, compose the RGB optical pose into the calibrated URDF, and retain it during regeneration. Add a ROS 2 Humble sensor TF process that uses RealSense internal extrinsics and a Jetson tmux bringup entrypoint.

No additional tests, builds, runtime launches, or post-work verification were performed, per workspace instructions.

File: SW/simulation/robot_description/robocup.calibrated.urdf (robot description, URDF)
Before this commit: robot robocup, 95 links, 94 joints
Joints:
- joint camera_link_joint: origin xyz=-0.1231374351388152 -0.00046627446244331891 1.2602505470202274 rpy=0.0041075243142279123 0.25740565260292736 0.0015486552345582768 -> xyz=-0.14374646438775088 0.026947328083129878 1.2634639227319704 rpy=-0.016534346952430324 0.229703005248273 0.0022884913799309371
