Commit message: feat(calibration): apply physical G2, Mid-360 and koide3 Head calibrations to Jetson
- Use selected Fusion 15 degree head camera mount as the default robot model
- Apply physical G2 calibration against Mid-360S to the calibrated URDF
- Address cross-review of the physical G2 calibration
- Apply accepted koide3 Head–Mid360 calibration and Jetson sensor TF
- Apply committed physical calibrations to Jetson robot bringup

Co-authored-by: kimsh039 <projectsh039@inha.edu>
Co-Authored-By: Claude Opus 5.5 <noreply@anthropic.com>

File: SW/simulation/robot_description/robocup.calibrated.urdf (robot description, URDF)
Before this commit: robot robocup, 95 links, 94 joints
Links:
- link rack_base_link: mass 15.6463681034 -> 15.6921304573; geometry collision box size=0.04 0.04 0.04; collision box size=0.04 0.04 0.04
Joints:
- joint cad_D435f_Solid_v1_1_joint: origin xyz=-0.12495 -2.611244554e-15 1.27 rpy=1.57079632679 1.25108409187e-29 1.57079632679 -> xyz=-0.120666319792 0.00125 1.26068901712 rpy=1.83259571459 1.2669865157e-12 1.57079632679
- joint camera_link_joint: origin xyz=-0.12722342972197517 -0.001716274462443348 1.2689368986951095 rpy=0.0037066991262989625 -0.0043934350517067511 0.0014976471610455334 -> xyz=-0.14374646438775088 0.026947328083129878 1.2634639227319704 rpy=-0.016534346952430324 0.229703005248273 0.0022884913799309371
- joint laser_frame_joint: origin xyz=-5.1389834908760446e-05 0.00052051635559500814 0 rpy=0 0 0.15437059215843318 -> xyz=0.024073172308992453 0.0091594372740952668 0 rpy=0 0 0.049509674634016343
- joint livox_frame_joint: origin xyz=3.773355003483525e-05 0.00015620113972823895 -0.00024318079626794997 rpy=3.1415281256409191 2.0508080655012861e-05 -2.7091518517208257e-05 -> xyz=3.773355003483525e-05 0.00015620113972823895 -0.00024318079626794997 rpy=3.1415281256409195 2.0508080655234906e-05 -2.7091518517184195e-05
- joint piper_to_wrist_camera_mount: origin xyz=0.00021057778731321184 0.00081284728291651563 0.0072422552841638725 rpy=-1.5721318918257796 -0.0019379665882315322 1.6152889735146658 -> xyz=0.00021057778731321808 0.00081284728291651596 0.0072422552841638725 rpy=-1.5721318918257798 -0.0019379665882315322 1.6152889735146665
